File: RF-AMP-VHF_V1.kicad_pcb (KiCad board)
At the start: 2 copper layers, 180 x 120 mm, 123 parts, among them J1 DB15_Male, J2 RF IN, J3 RF OUT, Q1 BC857, Q2 BLF189XRA, Q3 BC847, U1 L78L05_SOT89, U2 L79L05_SOT89, U3 LM7332, U4 TMP36GT9

Commit message: initial commit
Parts:
- removed the D2 at (175.6, -6.92)
- removed the D4 at (91.1, 18.1)
- removed D9: BAT54W, Package_TO_SOT_SMD:SOT-323_SC-70
- removed the J1 at (25.0, 132.0)
- added C60: 100n, Capacitor_SMD:C_0805_2012Metric, F.Cu at (92.5, 133.2)
- added C61: 100n, Capacitor_SMD:C_0805_2012Metric, F.Cu at (89.0, 144.8)
- added C62: 22p, Capacitor_SMD:C_1210_3225Metric, F.Cu at (52.5, 67.0)
- added D3: 1N4148W, Diode_SMD:D_SOD-123, F.Cu at (74.8, 129.5)
- added D5: BAT54SW, Package_TO_SOT_SMD:SOT-323_SC-70, F.Cu at (202.0, 85.9)
- added FB4: BLM21BD102, Resistor_SMD:R_0805_2012Metric, F.Cu at (88.0, 130.0)
- added FB5: BLM21BD102, Resistor_SMD:R_0805_2012Metric, F.Cu at (98.0, 126.5)
- added J3: RF IN ATT, Connector_Coaxial:SMA_Amphenol_132289_EdgeMount, F.Cu at (38.0, 64.5)
- added L9: 22n, Inductor_SMD:L_Neosid_Air-Coil_SML_3turn_HDM0331A, F.Cu at (52.8, 73.8)
- added R30: 100, Package_TO_SOT_SMD:TO-263-2, F.Cu at (63.0, 53.0)
- added R31: 68, Package_TO_SOT_SMD:TO-263-2, F.Cu at (63.0, 67.0)
- added R32: 100, Package_TO_SOT_SMD:TO-263-2, F.Cu at (63.0, 81.0)
- added REF**: MountingHole_3.2mm_M3_Pad, MountingHole:MountingHole_3.2mm_M3_Pad, F.Cu at (76.0, 67.0)
- added REF**: MountingHole_4.3mm_M4_Pad, MountingHole:MountingHole_4.3mm_M4_Pad, F.Cu at (97.2, 153.0)
- added REF**: MountingHole_4.3mm_M4_Pad, MountingHole:MountingHole_4.3mm_M4_Pad, F.Cu at (122.8, 153.0)
- added REF**: MountingHole_4.3mm_M4_Pad, MountingHole:MountingHole_4.3mm_M4_Pad, F.Cu at (122.8, 125.0)
- added REF**: MountingHole_4.3mm_M4_Pad, MountingHole:MountingHole_4.3mm_M4_Pad, F.Cu at (122.8, 75.0)
- added REF**: MountingHole_4.3mm_M4_Pad, MountingHole:MountingHole_4.3mm_M4_Pad, F.Cu at (122.8, 47.0)
- added REF**: MountingHole_4.3mm_M4_Pad, MountingHole:MountingHole_4.3mm_M4_Pad, F.Cu at (97.2, 47.0)
- added REF**: MountingHole_3.2mm_M3_Pad, MountingHole:MountingHole_3.2mm_M3_Pad, F.Cu at (76.0, 53.0)
- added REF**: MountingHole_3.2mm_M3_Pad, MountingHole:MountingHole_3.2mm_M3_Pad, F.Cu at (183.0, 85.0)
- added REF**: MountingHole_3.2mm_M3_Pad, MountingHole:MountingHole_3.2mm_M3_Pad, F.Cu at (183.0, 115.0)
- added REF**: MountingHole_3.2mm_M3_Pad, MountingHole:MountingHole_3.2mm_M3_Pad, F.Cu at (40.0, 85.0)
- added REF**: MountingHole_3.2mm_M3_Pad, MountingHole:MountingHole_3.2mm_M3_Pad, F.Cu at (40.0, 115.0)
- added REF**: MountingHole_3.2mm_M3_Pad, MountingHole:MountingHole_3.2mm_M3_Pad, F.Cu at (219.5, 115.0)
- added REF**: MountingHole_3.2mm_M3_Pad, MountingHole:MountingHole_3.2mm_M3_Pad, F.Cu at (219.5, 85.0)
- C57, C58: value 1n -> 330p
- D1, D6, D7, D8: value BAT54W -> BAT54SW
- L2: footprint Inductor_SMD:L_Neosid_Air-Coil_SML_6-10turn_HDM0431A-HDM1031A -> RF-AMP-VHF_V1:L_Neosid_Air-Coil_SML_6-10turn_HDM0431A-HDM1031A
- L3, L4, L5, L6, L7: footprint Inductor_SMD:L_Neosid_Air-Coil_SML_6-10turn_HDM0431A-HDM1031A -> RF-AMP-VHF_V1:Air_Coil_1
- L8: value L -> 22n; footprint Inductor_SMD:L_Neosid_Air-Coil_SML_6-10turn_HDM0431A-HDM1031A -> Inductor_SMD:L_Neosid_Air-Coil_SML_3turn_HDM0331A
- REF** (x4): value MountingHole_5.3mm_M5_Pad -> MountingHole_4.3mm_M4_Pad; footprint MountingHole:MountingHole_5.3mm_M5_Pad -> MountingHole:MountingHole_4.3mm_M4_Pad
- U4: footprint Package_SO:SOIC-8_3.9x4.9mm_P1.27mm -> Package_TO_SOT_THT:TO-92_Inline_W4.0mm_Horizontal_FlatSideDown
- moved C2 230.5 mm to (53.5, 144.8), turned to 270 degrees
- moved C7 222.9 mm to (60.8, 144.8), turned to 90 degrees
- moved C4 219.3 mm to (56.5, 144.8), turned to 270 degrees
- moved U1 210.4 mm to (66.5, 135.0), turned to 270 degrees
- moved FB2 209.0 mm to (55.0, 142.0), turned to 180 degrees
- moved C24 204.7 mm to (86.3, 139.0), turned to 90 degrees
- moved C10 204.1 mm to (55.5, 102.5), turned to 270 degrees
- moved FB3 203.2 mm to (47.8, 113.5), turned to 270 degrees
- moved R13 200.3 mm to (96.5, 143.5), turned to 270 degrees
- moved C8 197.3 mm to (48.8, 102.0), turned to 270 degrees
- moved RV1 196.3 mm to (77.5, 140.0), turned to 90 degrees
- moved C11 196.2 mm to (70.2, 134.5), turned to 270 degrees
- moved C12 193.7 mm to (70.2, 144.5), turned to 90 degrees
- moved R15 190.7 mm to (95.8, 138.2), turned to 270 degrees
- moved C18 190.6 mm to (79.5, 100.0), turned to 270 degrees
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- renumbered C9 to C8, C8 to C9, D3 to D2, D5 to D4, J2 to J1, J3 to J2
Connections:
- C1 pad 1: Net-(C1-Pad1) -> +12V
- C2 pad 1: Net-(C2-Pad1) -> -12V
- C27 pad 1: GATE -> Net-(C27-Pad1)
- C3 pad 1: +12V -> Net-(C3-Pad1)
- C38 pad 1: GATE -> Net-(C27-Pad1)
- C4 pad 1: -12V -> Net-(C4-Pad1)
- C6 pad 1: +12V -> Net-(C3-Pad1)
- C7 pad 2: -12V -> Net-(C4-Pad1)
- C8 pad 2: Net-(C9-Pad2) -> Net-(C8-Pad2)
- C9 pad 1: Net-(C8-Pad1) -> Net-(C10-Pad1)
- C9 pad 2: Net-(C10-Pad1) -> Net-(C9-Pad2)
- D1 pad 1: Net-(C8-Pad1) -> Net-(C9-Pad2)
- D1 pad 2: Net-(D1-Pad2) -> Net-(C8-Pad2)
- D6 pad 3: Net-(C56-Pad1) -> Earth
- D8 pad 1: Net-(D8-Pad1) -> Earth
- D8 pad 2: Net-(D8-Pad2) -> Net-(C59-Pad1)
- D8 pad 3: Earth -> Net-(D8-Pad3)
- FB1 pad 1: +12V -> Net-(C3-Pad1)
- FB1 pad 2: Net-(C1-Pad1) -> +12V
- FB2 pad 1: -12V -> Net-(C4-Pad1)
- FB2 pad 2: Net-(C2-Pad1) -> -12V
- J2 pad 1: Net-(J3-Pad1) -> Net-(C55-Pad1)
- L2 pad 1: Net-(C16-Pad1) -> Net-(L1-Pad2)
- L2 pad 2: Net-(L1-Pad2) -> Net-(C16-Pad1)
- L8 pad 1: Net-(C55-Pad1) -> Net-(C62-Pad2)
- L8 pad 2: Net-(J3-Pad1) -> Net-(L8-Pad2)
- R11 pad 2: Net-(C23-Pad1) -> Net-(FB5-Pad2)
- R12 pad 2: Net-(C23-Pad1) -> Net-(FB5-Pad2)
- R14 pad 1: GATE -> Net-(C27-Pad1)
- R2 pad 1: Net-(C9-Pad2) -> Net-(C8-Pad2)
- R20 pad 1: Net-(D6-Pad1) -> Net-(D5-Pad3)
- R21 pad 2: Net-(D7-Pad1) -> Net-(D6-Pad1)
- R22 pad 2: Net-(D6-Pad1) -> Net-(D5-Pad3)
- R25 pad 1: Net-(D9-Pad1) -> Net-(D8-Pad3)
- R26 pad 2: Net-(D8-Pad1) -> Net-(D7-Pad1)
- R27 pad 1: Net-(D9-Pad1) -> Net-(D8-Pad3)
- U1 pad 3: +12V -> Net-(C3-Pad1)
- U2 pad 2: -12V -> Net-(C4-Pad1)
- U3 pad 1: GATE -> Net-(C27-Pad1)
Routing:
- net +5V: track 0.00 -> 61.5 mm
- net TEMP: track 0.00 -> 38.5 mm
- net -5V: track 0.00 -> 34.3 mm
- net Net-(C62-Pad1): track 0.00 -> 33.0 mm
- net GATE: track 0.00 -> 30.3 mm
- net Net-(C55-Pad1): track 0.00 -> 29.2 mm
- net Net-(C62-Pad2): track 0.00 -> 19.2 mm
- net Net-(FB5-Pad2): track 0.00 -> 18.7 mm
- net Net-(C10-Pad1): track 0.00 -> 17.5 mm
- net Net-(C4-Pad1): track 0.00 -> 16.7 mm
- net GATE_EN: track 0.00 -> 15.4 mm
- net Net-(D4-Pad1): track 0.00 -> 12.8 mm
- net Net-(C3-Pad1): track 0.00 -> 11.8 mm
- net Net-(C24-Pad1): track 0.00 -> 11.5 mm
- net Net-(C24-Pad2): track 0.00 -> 10.7 mm
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- added copper zone on F.Cu, net (none)
- added copper zone on F.Cu, net +12V
- added copper zone on F.Cu, net -12V
- added copper zone on B.Cu, net Earth
- added copper zone on F.Cu, net Earth
- added copper zone on F.Cu, net FWD
- added copper zone on F.Cu, net GATE_EN
- added copper zone on F.Cu, net Net-(C10-Pad1)
- added copper zone on F.Cu, net Net-(C16-Pad1)
- added copper zone on F.Cu, net Net-(C16-Pad2)
- added copper zone on F.Cu, net Net-(C17-Pad1)
- added copper zone on F.Cu, net Net-(C17-Pad2)
- added copper zone on F.Cu, net Net-(C21-Pad1)
- added copper zone on F.Cu, net Net-(C22-Pad1)
- added copper zone on F.Cu, net Net-(C25-Pad1)
- added copper zone on F.Cu, net Net-(C25-Pad2)
- added copper zone on F.Cu, net Net-(C28-Pad2)
- added copper zone on F.Cu, net Net-(C32-Pad2)
- added copper zone on F.Cu, net Net-(C39-Pad1)
- added copper zone on F.Cu, net Net-(C42-Pad1)
- added copper zone on F.Cu, net Net-(C52-Pad1)
- added copper zone on F.Cu, net Net-(C53-Pad1)
- added copper zone on F.Cu, net Net-(C54-Pad1)
- added copper zone on F.Cu, net Net-(C55-Pad1)
- added copper zone on F.Cu, net Net-(L1-Pad2)
- added copper zone on F.Cu, net Net-(L8-Pad2)
- added copper zone on F.Cu, net Net-(L9-Pad2)
- added copper zone on F.Cu, net Net-(Q2-Pad1)
- added copper zone on F.Cu, net Net-(Q2-Pad2)
- added copper zone on F.Cu, net Net-(Q2-Pad3)
- added copper zone on F.Cu, net Net-(Q2-Pad4)
- added copper zone on F.Cu, net Net-(R18-Pad1)
- added copper zone on F.Cu, net Net-(R22-Pad1)
- added copper zone on F.Cu, net REF
- added copper zone on F.Cu, net RF_OL
- added copper zone on F.Cu, net TEMP
- added copper zone on F.Cu, net VDD
Other:
- board size 180 x 120 mm -> 190 x 120 mm
- net class RF1 added: clearance 1.5, trace_width 3.37, via_dia 0.8, via_drill 0.4
- board text added: "+12V"
- board text added: "-12V"
- board text added: "GATE_EN"
- board text added: "RF_OL"
- board text added: "TEMP"

Commit message: initial commit
Parts:
- added REF**: KiCad-Logo2_6mm_SilkScreen, Symbol:KiCad-Logo2_6mm_SilkScreen, F.Cu at (90.5, 55.0)
Routing:
- added copper zone on F.Cu, net Net-(C62-Pad1)
Other:
- board text added: "FWD"
- board text added: "HB9GKW LDMOS_RF_AMP_V1"
- board text added: "REF"
- board text added: "VDD"
