File: RF-AMP-VHF_V1.kicad_pcb (KiCad board)
At the start: 2 copper layers, 190 x 120 mm, 146 parts, among them J1 RF IN, J2 RF OUT, J3 RF IN ATT, Q1 BC857, Q2 BLF189XRA, Q3 BC847, U1 L78L05_SOT89, U2 L79L05_SOT89, U3 LM7332, U4 TMP36GT9

Commit message: changing gerber format
Routing:
- net Earth: vias 701 -> 699
Changed lines of the file:
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@@
-(kicad_pcb (version 20171130) (host pcbnew 5.1.5+dfsg1-2~bpo10+1)
+(kicad_pcb (version 20171130) (host pcbnew "(5.1.5)-3")
   (general
     (thickness 1.6)
     (drawings 56)
-    (tracks 899)
+    (tracks 897)
     (zones 0)
     (modules 146)
@@
     (solder_mask_min_width 0.25)
     (aux_axis_origin 0 0)
-    (visible_elements FFFFFF7F)
+    (visible_elements 7FFFFFFF)
     (pcbplotparams
       (layerselection 0x010e0_ffffffff)
@@
   (via (at 193.25 73.05) (size 0.8) (drill 0.4) (layers F.Cu B.Cu) (net 1))
   (via (at 196.25 73.05) (size 0.8) (drill 0.4) (layers F.Cu B.Cu) (net 1))
-  (via (at 152.75 75.85) (size 0.8) (drill 0.4) (layers F.Cu B.Cu) (net 1))
   (via (at 155.75 75.85) (size 0.8) (drill 0.4) (layers F.Cu B.Cu) (net 1))
   (via (at 158.75 75.85) (size 0.8) (drill 0.4) (layers F.Cu B.Cu) (net 1))
@@
   (via (at 193.25 78.65) (size 0.8) (drill 0.4) (layers F.Cu B.Cu) (net 1))
   (via (at 196.25 78.65) (size 0.8) (drill 0.4) (layers F.Cu B.Cu) (net 1))
-  (via (at 152.75 81.45) (size 0.8) (drill 0.4) (layers F.Cu B.Cu) (net 1))
   (via (at 155.75 81.45) (size 0.8) (drill 0.4) (layers F.Cu B.Cu) (net 1))
   (via (at 158.75 81.45) (size 0.8) (drill 0.4) (layers F.Cu B.Cu) (net 1))

Commit message: Review 1
Routing:
- net Earth: vias 699 -> 570
