File: RF-AMP-VHF_V1.kicad_pcb (KiCad board)
At the start: 2 copper layers, 190 x 120 mm, 146 parts, among them J1 RF IN, J2 RF OUT, J3 RF IN ATT, Q1 BC857, Q2 BLF189XRA, Q3 BC847, U1 L78L05_SOT89, U2 L79L05_SOT89, U3 LM7332, U4 TMP36GT9

Commit message: prototype release
Routing:
- net Earth: vias 570 -> 569
Changed lines of the file:
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@@
-(kicad_pcb (version 20171130) (host pcbnew "(5.1.5)-3")
+(kicad_pcb (version 20171130) (host pcbnew 5.1.5+dfsg1-2~bpo10+1)
   (general
     (thickness 1.6)
     (drawings 56)
-    (tracks 768)
+    (tracks 767)
     (zones 0)
     (modules 146)
@@
   (via (at 101.75 84.25) (size 1.5) (drill 1) (layers F.Cu B.Cu) (net 1))
   (via (at 101.75 81.25) (size 1.5) (drill 1) (layers F.Cu B.Cu) (net 1))
-  (via (at 197.75 70.25) (size 1.5) (drill 1) (layers F.Cu B.Cu) (net 1))
   (segment (start 53.5 132.0625) (end 54.0625 131.5) (width 1) (layer F.Cu) (net 2))
   (segment (start 53.5 133.3125) (end 53.5 132.0625) (width 1) (layer F.Cu) (net 2))

Commit message: bug fixes
Parts:
- D2: value BZX84C33 -> BZX84C5V6
- D4: value BZX84C33 -> BZX84C3V3
- moved C55 4.25 mm to (193.2, 97.0)
- moved R10 2.84 mm to (83.5, 142.0), turned to 180 degrees
- moved C24 1.80 mm to (86.3, 140.8), turned to 270 degrees
- moved C52 1.75 mm to (172.2, 97.0)
Connections:
- C24 pad 2: Net-(C24-Pad2) -> Earth
- C27 pad 2: Net-(C24-Pad2) -> Net-(C27-Pad2)
- R11 pad 1: Net-(C24-Pad2) -> Net-(C27-Pad2)
- R14 pad 2: Net-(C24-Pad2) -> Net-(C27-Pad2)
- U3 pad 2: Net-(C24-Pad2) -> Net-(C27-Pad2)
Routing:
- net Net-(C27-Pad2): track 0.00 -> 10.7 mm
- net Net-(C24-Pad2): track 10.7 -> 0.00 mm
- net Net-(C24-Pad1): track 11.5 -> 12.0 mm

Commit message: prototype improvements
Parts:
- added R33: 10k, Resistor_SMD:R_0805_2012Metric, F.Cu at (76.2, 131.0)
- C24: value 100n -> 1n
- C53, C54: value 1p8 -> 27p
- C8, C9: value 1p8 -> 6p8
- D4: value BZX84C3V3 -> BZX84C5V6
- L1, L2: value 820n -> 150n
- L3, L4: value L -> 330n
- L5, L7: value L -> 61n
- L6: value L -> 105n
- R7, R8: value 47k -> 4k7
- moved D3 5.20 mm to (69.6, 129.5)
- moved R7 1.50 mm to (73.2, 131.0), turned to 90 degrees
Connections:
- L3 pad 2: Net-(C28-Pad2) -> Net-(C32-Pad2)
- L4 pad 1: Net-(C32-Pad2) -> Net-(C28-Pad2)
- Q2 pad 1: Net-(Q2-Pad1) -> Net-(C32-Pad2)
- Q2 pad 2: Net-(Q2-Pad2) -> Net-(C28-Pad2)
Routing:
- net GATE_EN: track 15.4 -> 10.2 mm
- net Net-(D3-Pad1): track 4.48 -> 7.99 mm
- net Net-(D2-Pad2): track 1.57 -> 3.38 mm
- removed copper zone on F.Cu, net Net-(Q2-Pad1)
- removed copper zone on F.Cu, net Net-(Q2-Pad2)

Commit message: prototype improvements
Parts:
- R33: value 10k -> 4k7
- R8: value 4k7 -> 47k
Changed lines of the file:
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@@
   )
   (setup
-    (last_trace_width 0.5)
+    (last_trace_width 0.25)
     (user_trace_width 0.5)
     (user_trace_width 0.75)
@@
       (effects (font (size 1 1) (thickness 0.15)))
     )
-    (fp_text value 4k7 (at 0 1.65 90) (layer F.Fab)
+    (fp_text value 47k (at 0 1.65 90) (layer F.Fab)
       (effects (font (size 1 1) (thickness 0.15)))
     )
@@
       (effects (font (size 1 1) (thickness 0.15)))
     )
-    (fp_text value 10k (at 0 1.65 90) (layer F.Fab)
+    (fp_text value 4k7 (at 0 1.65 90) (layer F.Fab)
       (effects (font (size 1 1) (thickness 0.15)))
     )
